Commit message: Testing again without sourcing other catkin_ws

File: antobot_descriptions/antobot_ant_description/urdf/ant.urdf.xacro (robot description, xacro)
@@ -15,9 +15,9 @@
 # OF THIS SOFTWARE, EVEN IF ADVISED OF THE POSSIBILITY OF SUCH DAMAGE.
 # # # # # # # # # # # # # # # # # # # # # # # # # # # # # # # # # # # # # # # # # # # # # # # # # # # # # # # # # # # # #
-# # # Code Description:     URDF for AntoBot VP1
+# # # Code Description:     URDF for AntoBot Ant
 # Contact: william.eaton@antobot.ai
 # # # #  # # # # # # # # # # # # # # # # # # # # # # # # # # # # # # # # # # # # # # # # # # # # # # # # # # # # # # # # #
 -->
-<robot name="antobot_vp1" xmlns:xacro="http://ros.org/wiki/xacro">
+<robot name="antobot_ant" xmlns:xacro="http://ros.org/wiki/xacro">
   <!-- Arguments -->
   <xacro:arg name="zed2_orientation"   default="left" />
@@ -28,5 +28,5 @@
   <xacro:property name="referenceLongitude"    value="$(arg referenceLongitude)" />
   <!-- antobot -->
-  <xacro:macro name="antobot_vp1">
+  <xacro:macro name="antobot_ant_description">
     <xacro:property name="M_PI" value="3.1415926535897931" />
     <link name="base_link" />
@@ -34,5 +34,5 @@
       <visual>
         <geometry>
-          <mesh filename="package://antobot_vp1/meshes/chassis.dae" scale="1 1 1"/>
+          <mesh filename="package://antobot_ant_description/meshes/chassis.dae" scale="1 1 1"/>
         </geometry>
         <origin xyz="0 0 0" rpy="0 0 0"/>
@@ -40,5 +40,5 @@
       <collision>
        <geometry>
-          <mesh filename="package://antobot_vp1/meshes/chassis.dae" scale="1 1 1"/>
+          <mesh filename="package://antobot_ant_description/meshes/chassis.dae" scale="1 1 1"/>
         </geometry>
         <origin xyz="0 0 0" rpy="0 0 0"/>
@@ -68,5 +68,5 @@
       <visual>
         <geometry>
-          <mesh filename="package://antobot_vp1/meshes/wheel.dae" scale="1 1 1" />
+          <mesh filename="package://antobot_ant_description/meshes/wheel.dae" scale="1 1 1" />
         </geometry>
         <origin xyz="0 0 0" rpy="0 0 ${M_PI}"/>
@@ -97,5 +97,5 @@
       <visual>
         <geometry>
-          <mesh filename="package://antobot_vp1/meshes/wheel.dae" scale="1 1 1" />
+          <mesh filename="package://antobot_ant_description/meshes/wheel.dae" scale="1 1 1" />
         </geometry>
         <origin xyz="0 0 0" rpy="0 0 ${M_PI}"/>
@@ -126,5 +126,5 @@
       <visual>
         <geometry>
-          <mesh filename="package://antobot_vp1/meshes/wheel.dae" scale="1 1 1" />
+          <mesh filename="package://antobot_ant_description/meshes/wheel.dae" scale="1 1 1" />
         </geometry>
         <origin xyz="0 0 0" rpy="0 0 0"/>
@@ -155,5 +155,5 @@
       <visual>
         <geometry>
-          <mesh filename="package://antobot_vp1/meshes/wheel.dae" scale="1 1 1" />
+          <mesh filename="package://antobot_ant_description/meshes/wheel.dae" scale="1 1 1" />
         </geometry>
         <origin xyz="0 0 0" rpy="0 0 0"/>
@@ -269,10 +269,10 @@
 	  <origin xyz="0 0 0" rpy="0 0 0" />
 	  <geometry>
-      <mesh filename="package://antobot_vp1/meshes/rpLidar.dae" scale="1 1 1" />
+      <mesh filename="package://antobot_ant_description/meshes/rpLidar.dae" scale="1 1 1" />
 	  </geometry>
 	</collision>
   <visual>
     <geometry>
-      <mesh filename="package://antobot_vp1/meshes/rpLidar.dae" scale="1 1 1" />
+      <mesh filename="package://antobot_ant_description/meshes/rpLidar.dae" scale="1 1 1" />
     </geometry>
     <origin xyz="0 0 0" rpy="0 0 0"/>
@@ -415,19 +415,19 @@
   <!-- Ultrasonics-->
   <!-- Actual sensors output on combined topic /antobridge/uss_dist -->
-  <xacro:include filename="$(find antobot_vp1)/urdf/ultrasonic.urdf.xacro"/>
+  <xacro:include filename="$(find antobot_ant_description)/urdf/ultrasonic.urdf.xacro"/>
   <xacro:ultrasonic id="1" xyz="0.5355 0.317 0.282" rpy="0 0 0.785398" />
-  <xacro:include filename="$(find antobot_vp1)/urdf/ultrasonic.urdf.xacro"/>
+  <xacro:include filename="$(find antobot_ant_description)/urdf/ultrasonic.urdf.xacro"/>
   <xacro:ultrasonic id="2" xyz="0.66 0 0.2935" rpy="0 0 0" />
-  <xacro:include filename="$(find antobot_vp1)/urdf/ultrasonic.urdf.xacro"/>
+  <xacro:include filename="$(find antobot_ant_description)/urdf/ultrasonic.urdf.xacro"/>
   <xacro:ultrasonic id="3" xyz="0.5535 -0.317 0.282" rpy="0 0 -0.785398" />
-  <xacro:include filename="$(find antobot_vp1)/urdf/ultrasonic.urdf.xacro"/>
+  <xacro:include filename="$(find antobot_ant_description)/urdf/ultrasonic.urdf.xacro"/>
   <xacro:ultrasonic id="4" xyz="-0.0165 -0.3385 0.282" rpy="0 0 -1.5708" />
-  <xacro:include filename="$(find antobot_vp1)/urdf/ultrasonic.urdf.xacro"/>
+  <xacro:include filename="$(find antobot_ant_description)/urdf/ultrasonic.urdf.xacro"/>
   <xacro:ultrasonic id="5" xyz="-0.5685 -0.317 0.282" rpy="0 0 -2.35619" />
-  <xacro:include filename="$(find antobot_vp1)/urdf/ultrasonic.urdf.xacro"/>
+  <xacro:include filename="$(find antobot_ant_description)/urdf/ultrasonic.urdf.xacro"/>
   <xacro:ultrasonic id="6" xyz="-0.5899 0 0.2878" rpy="0 0 3.14159" />
-  <xacro:include filename="$(find antobot_vp1)/urdf/ultrasonic.urdf.xacro"/>
+  <xacro:include filename="$(find antobot_ant_description)/urdf/ultrasonic.urdf.xacro"/>
   <xacro:ultrasonic id="7" xyz="-0.5685 0.317 0.282" rpy="0 0 2.35619" />
-  <xacro:include filename="$(find antobot_vp1)/urdf/ultrasonic.urdf.xacro"/>
+  <xacro:include filename="$(find antobot_ant_description)/urdf/ultrasonic.urdf.xacro"/>
   <xacro:ultrasonic id="8" xyz="-0.0165 0.3385 0.282" rpy="0 0 1.5708" />
   <!-- ZED camera -->
@@ -446,11 +446,11 @@
       <visual>
         <geometry>
-          <mesh filename="package://antobot_vp1/meshes/zedMountLeft.dae" scale="1 1 1" />
-        </geometry>
-        <origin xyz="0 0 0" rpy="0 0 0"/>
-      </visual>
-      <collision>
-        <geometry>
-          <mesh filename="package://antobot_vp1/meshes/zedMountLeft.dae" scale="1 1 1" />
+          <mesh filename="package://antobot_ant_description/meshes/zedMountLeft.dae" scale="1 1 1" />
+        </geometry>
+        <origin xyz="0 0 0" rpy="0 0 0"/>
+      </visual>
+      <collision>
+        <geometry>
+          <mesh filename="package://antobot_ant_description/meshes/zedMountLeft.dae" scale="1 1 1" />
         </geometry>
         <origin xyz="0 0 0" rpy="0 0 0"/>
@@ -476,11 +476,11 @@
       <visual>
         <geometry>
-          <mesh filename="package://antobot_vp1/meshes/zedMountLeft.dae" scale="1 1 1" />
-        </geometry>
-        <origin xyz="0 0 0" rpy="0 0 0"/>
-      </visual>
-      <collision>
-        <geometry>
-          <mesh filename="package://antobot_vp1/meshes/zedMountLeft.dae" scale="1 1 1" />
+          <mesh filename="package://antobot_ant_description/meshes/zedMountLeft.dae" scale="1 1 1" />
+        </geometry>
+        <origin xyz="0 0 0" rpy="0 0 0"/>
+      </visual>
+      <collision>
+        <geometry>
+          <mesh filename="package://antobot_ant_description/meshes/zedMountLeft.dae" scale="1 1 1" />
         </geometry>
         <origin xyz="0 0 0" rpy="0 0 0"/>
@@ -506,11 +506,11 @@
       <visual>
         <geometry>
-          <mesh filename="package://antobot_vp1/meshes/zedMountRight.dae" scale="1 1 1" />
-        </geometry>
-        <origin xyz="0 0 0" rpy="0 0 0"/>
-      </visual>
-      <collision>
-        <geometry>
-          <mesh filename="package://antobot_vp1/meshes/zedMountRight.dae" scale="1 1 1" />
+          <mesh filename="package://antobot_ant_description/meshes/zedMountRight.dae" scale="1 1 1" />
+        </geometry>
+        <origin xyz="0 0 0" rpy="0 0 0"/>
+      </visual>
+      <collision>
+        <geometry>
+          <mesh filename="package://antobot_ant_description/meshes/zedMountRight.dae" scale="1 1 1" />
         </geometry>
         <origin xyz="0 0 0" rpy="0 0 0"/>
@@ -543,5 +543,5 @@
   </joint>
   <link name="scouting_frame_right"/>
-  <xacro:include filename="$(find antobot_vp1)/urdf/zed2.urdf.xacro"/>
+  <xacro:include filename="$(find antobot_ant_description)/urdf/zed2.urdf.xacro"/>
   <xacro:zed2_front link_prefix=''
               joint_prefix=''/>
@@ -553,9 +553,9 @@
       <origin xyz="-0.676 -0.078 0.381" rpy="0 0 ${M_PI}"/>
   </joint>
-  <xacro:include filename="$(find antobot_vp1)/urdf/zed2_back.urdf.xacro"/>
+  <xacro:include filename="$(find antobot_ant_description)/urdf/zed2_back.urdf.xacro"/>
   <xacro:zed2_back link_prefix=''
                    joint_prefix=''/>
   <xacro:zed2_back_gazebo robot_ns=''/>
   </xacro:macro>
-  <xacro:antobot_vp1/>
+  <xacro:antobot_ant_description/>
 </robot>

File: antobot_descriptions/antobot_ant_description/urdf/zed2.urdf.xacro (robot description, xacro)
@@ -17,10 +17,10 @@
       <visual>
         <geometry>
-            <mesh filename="package://antobot_vp1/meshes/zed2.dae" scale="1 1 1" />
+            <mesh filename="package://antobot_ant_description/meshes/zed2.dae" scale="1 1 1" />
         </geometry>
       </visual>
       <collision>
         <geometry>
-            <mesh filename="package://antobot_vp1/meshes/zed2.dae" scale="1 1 1" />
+            <mesh filename="package://antobot_ant_description/meshes/zed2.dae" scale="1 1 1" />
         </geometry>
       </collision>

File: antobot_descriptions/antobot_ant_description/urdf/zed2_back.urdf.xacro (robot description, xacro)
@@ -17,10 +17,10 @@
       <visual>
         <geometry>
-            <mesh filename="package://antobot_vp1/meshes/zed2.dae" scale="1 1 1" />
+            <mesh filename="package://antobot_ant_description/meshes/zed2.dae" scale="1 1 1" />
         </geometry>
       </visual>
       <collision>
         <geometry>
-            <mesh filename="package://antobot_vp1/meshes/zed2.dae" scale="1 1 1" />
+            <mesh filename="package://antobot_ant_description/meshes/zed2.dae" scale="1 1 1" />
         </geometry>
       </collision>
