Commit message: Changed wheel collision from cyclinder to sphere to improve dynamics

File: antobot_descriptions/antobot_description/urdf/ant_wheel.urdf.xacro (robot description, xacro)
@@ -32,5 +32,5 @@
       <collision>
         <geometry>
-          <cylinder length="0.08" radius="0.16" />
+          <sphere radius="0.16" />
         </geometry>
         <origin xyz="0 ${centreOffset} 0" rpy="${M_PI/2} 0 0" />
