Commit message: Conversion to ROS2 - untested

File: antobot_descriptions/antobot_description/urdf/ant_v4.urdf.xacro (robot description, xacro)
@@ -9,11 +9,4 @@
 -->
 <robot name="antobot_ant" xmlns:xacro="http://ros.org/wiki/xacro">
-  <!-- Position for gazebo-->
-  <xacro:arg name="referenceLatitude"   default="51.45315122695476" />
-  <xacro:property name="referenceLatitude"    value="$(arg referenceLatitude)" />
-  <xacro:arg name="referenceLongitude"   default="-0.6079828525888944" />
-  <xacro:property name="referenceLongitude"    value="$(arg referenceLongitude)" />
-  <xacro:arg name="referenceHeading"   default="90.0" />
-  <xacro:property name="referenceHeading"    value="$(arg referenceHeading)" />
   <!-- Need argument to get from launch file -->
   <xacro:arg name="params_path" default="../config/platform_config.yaml"/>
@@ -60,45 +53,90 @@
     <xacro:ant_wheel name='right_front' originX='0.26' originY='-0.26' originZ='-0.013975' rotZ='0' centreOffset='-0.06'/>
     <gazebo>
-      <plugin name="gazebo_ros_control" filename="libgazebo_ros_control.so">
-        <robotNamespace>/</robotNamespace>
+      <plugin
+        filename="ignition-gazebo-diff-drive-system"
+        name="ignition::gazebo::systems::DiffDrive">
+        <left_joint>wheel_left_front_joint</left_joint>
+        <left_joint>wheel_left_rear_joint</left_joint>
+        <right_joint>wheel_right_front_joint</right_joint>
+        <right_joint>wheel_right_rear_joint</right_joint>
+        <wheel_separation>1.25</wheel_separation>
+        <wheel_radius>0.3</wheel_radius>
+        <odom_publish_frequency>1</odom_publish_frequency>
+        <publish_odom>true</publish_odom>
+        <odom_topic>/odom</odom_topic>
+        <odom_frame>odom</odom_frame>
+        <robot_base_frame>base_link</robot_base_frame>
+        <max_linear_acceleration>1</max_linear_acceleration>
+        <min_linear_acceleration>-1</min_linear_acceleration>
+        <max_angular_acceleration>2</max_angular_acceleration>
+        <min_angular_acceleration>-2</min_angular_acceleration>
+        <max_linear_velocity>2.0</max_linear_velocity>
+        <min_linear_velocity>-2.0</min_linear_velocity>
+        <max_angular_velocity>1</max_angular_velocity>
+        <min_angular_velocity>-1</min_angular_velocity>
+      </plugin>
+      <plugin
+        filename="ignition-gazebo-joint-state-publisher-system"
+        name="ignition::gazebo::systems::JointStatePublisher">
       </plugin>
     </gazebo>
-    <!-- Gazebo ground truth-->
-    <gazebo>
-    <plugin name="p3d_base_controller" filename="libgazebo_ros_p3d.so">
-      <alwaysOn>true</alwaysOn>
-      <updateRate>10.0</updateRate>
-      <bodyName>base_link</bodyName>
-      <topicName>ground_truth/state</topicName>
-      <gaussianNoise>0.0</gaussianNoise>
-      <frameName>world</frameName>
-      <xyzOffset>0 0 0</xyzOffset>
-      <rpyOffset>0 0 0</rpyOffset>
-    </plugin>
-    </gazebo>
-    <xacro:property name="lidar_list" value="${mp['lidar']}" />
-    <!-- Leishen C16 front lidar -->
-    <xacro:if value="${'c16' in lidar_list}">
-      <xacro:include filename="$(find antobot_description)/urdf/c16.urdf.xacro"/>
-      <xacro:property name="location" value="${mp['lidar']['c16']['location']}" />
-      <xacro:c16 link_prefix='' joint_prefix='' position='${location}'/>
-      <xacro:c16_gazebo robot_ns='' position='${location}'/>
-      <joint name="lidar_c16_joint_${mp['lidar']['c16']['location']}" type="fixed">
+    <xacro:property name="role" value="${mp['robot_role']}" />
+    <xacro:if value="${role == 'UV'}">
+      <!-- UV Frame link -->
+      <link name="uvFrame">
+        <visual>
+          <geometry>
+            <mesh filename="package://antobot_description/meshes/uvFrame.dae" scale="1 1 1"/>
+          </geometry>
+          <origin xyz="0 0 0" rpy="0 0 0"/>
+        </visual>
+        <collision>
+        <geometry>
+            <mesh filename="package://antobot_description/meshes/uvFrame.dae" scale="1 1 1"/>
+          </geometry>
+          <origin xyz="0 0 0" rpy="0 0 0"/>
+        </collision>
+      </link>
+      <joint name="uvFrame_joint" type="fixed">
+        <origin xyz="0 0 0.01" rpy="0 0 0" />
         <parent link="robot_base_link"/>
-        <child link="laser_link_${mp['lidar']['c16']['location']}_static"/>
-        <!-- <origin xyz="0.615 0.145 0.427" rpy="0 0 3.15"/> --><!-- When mounted low, on the left of the robot head -->
-        <origin xyz="${mp['lidar']['c16']['px']} ${mp['lidar']['c16']['py']} ${mp['lidar']['c16']['pz']}" rpy="${mp['lidar']['c16']['r']} ${mp['lidar']['c16']['p']} ${mp['lidar']['c16']['y']}"/>
+        <child link="uvFrame" />
       </joint>
     </xacro:if>
-    <!-- Leishen C16 rear lidar -->
-    <xacro:if value="${'c16_2' in lidar_list}">
+    <!-- ROS2 Humble doesn't support xacro:for yet - use if statements instead -->
+    <xacro:property name="robot_hardware"  value="${mp['robot_hardware']}"/>
+    <xacro:property name="lidars" value="${mp['lidar']}" />
+    <!-- Lidar 1 -->
+    <xacro:if value="${1 in lidars}">
+      <xacro:property name="lidar1" value="${lidars[1]}"/>
+      <xacro:property name="type1" value="${lidar1['type']}"/>
+      <xacro:property name="device_id"  value="${lidar1['device_id']}"/>
+      <!-- Include URDF for that lidar type -->
       <xacro:include filename="$(find antobot_description)/urdf/c16.urdf.xacro"/>
-      <xacro:property name="location" value="${mp['lidar']['c16_2']['location']}" />
-      <xacro:c16 link_prefix='' joint_prefix='' position='${location}'/>
-      <xacro:c16_gazebo robot_ns='' position='${location}'/>
-      <joint name="c16_lidar_joint_${mp['lidar']['c16_2']['location']}" type="fixed">
+      <xacro:c16 link_prefix="" joint_prefix="" position="${device_id}" robot_hardware="${robot_hardware}"/>
+      <xacro:c16_gazebo robot_ns="" position="${device_id}"/>
+      <!-- Fixed transform for Lidar 1 -->
+      <joint name="lidar_${type1}_1_joint_${device_id}" type="fixed">
         <parent link="robot_base_link"/>
-        <child link="laser_link_${mp['lidar']['c16_2']['location']}_static"/>
-        <origin xyz="${mp['lidar']['c16_2']['px']} ${mp['lidar']['c16_2']['py']} ${mp['lidar']['c16_2']['pz']}" rpy="${mp['lidar']['c16_2']['r']} ${mp['lidar']['c16_2']['p']} ${mp['lidar']['c16_2']['y']}"/>
+        <child link="lidar_${device_id}_link"/>
+        <origin
+          xyz="${lidar1['px']} ${lidar1['py']} ${lidar1['pz']}"
+          rpy="${lidar1['r']} ${lidar1['p']} ${lidar1['y']}"/>
+      </joint>
+    </xacro:if>
+    <!-- Lidar 2 -->
+    <xacro:if value="${2 in lidars}">
+      <xacro:property name="lidar2" value="${lidars[2]}"/>
+      <xacro:property name="type2" value="${lidar2['type']}"/>
+      <xacro:property name="device_id"  value="${lidar2['device_id']}"/>
+      <xacro:include filename="$(find antobot_description)/urdf/c16.urdf.xacro"/>
+       <xacro:c16 link_prefix="" joint_prefix="" position="${device_id}" robot_hardware="${robot_hardware}"/>
+      <xacro:c16_gazebo robot_ns="" position="${device_id}"/>
+      <joint name="lidar_${type2}_2_joint_${device_id}" type="fixed">
+        <parent link="robot_base_link"/>
+        <child link="lidar_${device_id}_link"/>
+        <origin
+          xyz="${lidar2['px']} ${lidar2['py']} ${lidar2['pz']}"
+          rpy="${lidar2['r']} ${lidar2['p']} ${lidar2['y']}"/>
       </joint>
     </xacro:if>
@@ -116,21 +154,23 @@
       </inertial>
     </link>
-    <gazebo>
-      <plugin name="gazebo_ros_gps" filename="libhector_gazebo_ros_gps.so" >
-        <updateRate>4.0</updateRate>
-        <bodyName>robot_base_link</bodyName> <!-- GPS plugin in simulation is publishing gps topic in base_link position - affecting EKF -->
-        <frameId>robot_base_link</frameId>
-        <topicName>/antobot_gps</topicName>
-        <velocityTopicName>/am_gps_vel</velocityTopicName>
-        <referenceLatitude>${referenceLatitude}</referenceLatitude>
-        <referenceLongitude>${referenceLongitude}</referenceLongitude>
-        <referenceHeading>${referenceHeading}</referenceHeading>
-        <referenceAltitude>10</referenceAltitude>
-        <offset>0 0 0</offset>
-        <drift>0.0 0.0 0.0</drift>
-        <gaussianNoise>0.01 0.01 0.01</gaussianNoise>
-        <velocityDrift>0 0 0</velocityDrift>
-        <velocityGaussianNoise>0.5 0.5 0.5</velocityGaussianNoise>
-      </plugin>
+    <gazebo reference="gps_frame">
+      <sensor name="gps_sensor" type="gps">
+        <pose>0 0 1 0 0 0</pose> <!-- adjust height as needed -->
+        <gps>
+          <horizontal_position_accuracy>1.0</horizontal_position_accuracy>
+          <vertical_position_accuracy>1.5</vertical_position_accuracy>
+          <position_sensing>
+            <noise type="gaussian">
+              <mean>0.0</mean>
+              <stddev>0.5</stddev>
+            </noise>
+          </position_sensing>
+        </gps>
+        <plugin name="ignition::gazebo::systems::NavSat"
+                filename="ignition-gazebo-navsat-system">
+          <topic>/gps/fix</topic>
+          <frame_id>gps_frame</frame_id>
+        </plugin>
+      </sensor>
     </gazebo>
     <!-- imu -->
@@ -142,18 +182,24 @@
     <link name="imu_frame">
       <inertial>
+        <origin xyz="0 0 0" rpy="0 0 0" />
         <mass value="0.270" />
-        <origin xyz="0 0 0" rpy="0 0 0" />
-        <inertia ixx="2.632e-4" ixy="0" ixz="0" iyy="2.632e-4" iyz="0" izz="1.62e-4" />
+        <inertia ixx="0.0002632" ixy="0.0" ixz="0.0" iyy="0.0002632" iyz="0.0" izz="0.000162" />
       </inertial>
     </link>
-    <gazebo>
-      <plugin name="imu_plugin" filename="libgazebo_ros_imu.so">
-        <alwaysOn>true</alwaysOn>
-        <bodyName>imu_frame</bodyName>
-        <topicName>/imu/data</topicName>
-        <serviceName>imu_service</serviceName>
-        <gaussianNoise>0.0</gaussianNoise>
-        <updateRate>20.0</updateRate>
-      </plugin>
+    <gazebo reference="imu_frame">
+      <sensor type="imu" name="imu_sensor">
+        <always_on>true</always_on>
+        <update_rate>100.0</update_rate>
+        <visualize>true</visualize>
+        <imu>
+          <topic>/imu/data</topic>
+          <orientation_reference_frame>ENU</orientation_reference_frame>
+        </imu>
+        <plugin name="ignition::gazebo::systems::Imu"
+                filename="ignition-gazebo-imu-system">
+          <topic>/imu/data</topic>
+          <frame_id>imu_frame</frame_id>
+        </plugin>
+      </sensor>
     </gazebo>
     <!-- Ultrasonics-->

File: antobot_descriptions/antobot_description/urdf/ant_wheel.urdf.xacro (robot description, xacro)
@@ -74,4 +74,5 @@
       </collision>
     </gazebo>
+    <!--
     <transmission name="wheel_${name}_trans" type="SimpleTransmission">
       <type>transmission_interface/SimpleTransmission</type>
@@ -84,4 +85,5 @@
       </joint>
     </transmission>
+    -->
   </xacro:macro>
 </robot>

File: antobot_descriptions/antobot_description/urdf/c16.urdf.xacro (robot description, xacro)
@@ -4,15 +4,22 @@
                params="link_prefix:=''
                        joint_prefix:=''
-                       position:='front'">
+                       position:='front'
+                       robot_hardware:='False'">
     <!-- Lidar Center (Emission point) -->
-    <link name="laser_link_${position}_static">
+    <link name="lidar_${position}_link">
     </link>
     <joint name="c16_lidar_${position}_frame_joint" type="fixed">
-        <parent link="laser_link_${position}_static"/>
-        <child link="laser_link_${position}_frame"/>
-        <origin xyz="0 0 -0.046093" rpy="0 0 0"/>
+        <parent link="lidar_${position}_link"/>
+        <child link="lidar_${position}_frame"/>
+        <xacro:if value="${robot_hardware}">
+          <origin xyz="0 0 -0.046093" rpy="0 0 0"/>
+        </xacro:if>
+        <xacro:unless value="${robot_hardware}">
+            <origin xyz="0 0 -0.046093" rpy="0 0 3.14"/> <!-- The gpu_lidar sensor's lidar frame has to be 180 deg rotated  -->
+        </xacro:unless>
+        <!--origin xyz="0 0 -0.046093" rpy="0 0 3.14"/-->  <!-- The gpu_lidar sensor's lidar frame has to be 180 deg rotated  -->
     </joint>
     <!-- The lidar frame position - for visualisation -->
-    <link name="laser_link_${position}_frame">
+    <link name="lidar_${position}_frame">
       <inertial>
         <mass value="1.0"/>
@@ -42,40 +49,44 @@
       <xacro:property name="link_prefix" value="${robot_ns}/"/>
     </xacro:if>
-    <gazebo reference="laser_link_${position}_static">
-      <sensor type="ray" name="lidar_${position}">
-        <always_on>true</always_on>
-        <pose>0 0 0 0 0 0</pose>
-        <visualize>false</visualize>
-        <update_rate>5</update_rate>
-        <ray>
-          <scan>
-            <horizontal>
-              <samples>1000</samples>
-              <resolution>1</resolution>
-              <min_angle>0</min_angle>
-              <max_angle>6.28318</max_angle>
-            </horizontal>
-            <vertical>
-              <samples>16</samples>
-              <resolution>1</resolution>
-              <min_angle>-0.2618</min_angle>
-              <max_angle>0.2618</max_angle>
-            </vertical>
-          </scan>
-            <range>
-            <min>0.4</min>
-            <max>20</max>
-            <resolution>0.01</resolution>
-          </range>
-        </ray>
-        <plugin name="plugin_1" filename="libgazebo_ros_velodyne_laser.so">
-            <gaussianNoise>0.00</gaussianNoise>
-            <alwaysOn>true</alwaysOn>
-            <updateRate>5</updateRate>
-            <topicName>/lidar_${position}/lslidar_point_cloud</topicName>
-            <frameName>laser_link_${position}</frameName>
-        </plugin>
+    <gazebo reference="lidar_${position}_link">
+      <sensor name='lidar_${position}' type='gpu_lidar'>"
+          <pose relative_to='lidar_${position}_frame'>0 0 0 0 0 0</pose>
+          <ignition_frame_id>lidar_${position}_frame</ignition_frame_id>
+          <topic>/lidar_${position}/scan</topic>
+          <update_rate>10</update_rate>
+          <ray>
+              <scan>
+                  <horizontal>
+                      <samples>640</samples>
+                      <resolution>1</resolution>
+                      <min_angle>-3.15</min_angle>
+                      <max_angle>3.15</max_angle>
+                  </horizontal>
+                  <vertical>
+                      <samples>100</samples>
+                      <resolution>1</resolution>
+                      <min_angle>-0.25</min_angle>
+                      <max_angle>0.25</max_angle>
+                  </vertical>
+              </scan>
+              <range>
+                  <min>0.1</min>
+                  <max>20.0</max>
+                  <resolution>0.01</resolution>
+              </range>
+          </ray>
+          <always_on>1</always_on>
+          <visualize>true</visualize>
       </sensor>
     </gazebo>
   </xacro:macro>
 </robot>
+<!--
+<plugin name="plugin_1" filename="libgazebo_ros_velodyne_laser.so">
+    <gaussianNoise>0.00</gaussianNoise>
+    <alwaysOn>true</alwaysOn>
+    <updateRate>5</updateRate>
+    <topicName>/lidar_${position}/lslidar_point_cloud</topicName>
+    <frameName>laser_link_${position}</frameName>
+</plugin>
+-->

File: antobot_descriptions/antobot_description/urdf/ls_ch128x1.urdf.xacro (robot description, xacro)
@@ -77,4 +77,5 @@
           </range>
         </ray>
+        <!--
         <plugin name="plugin_1" filename="libgazebo_ros_velodyne_laser.so">
             <gaussianNoise>0.00</gaussianNoise>
@@ -84,4 +85,5 @@
             <frameName>laser_link_ch128_imu_${position}</frameName>
         </plugin>
+        -->
       </sensor>
     </gazebo>

File: antobot_descriptions/antobot_description/urdf/ultrasonic.urdf.xacro (robot description, xacro)
@@ -53,4 +53,5 @@
           </range>
         </ray>
+        <!--
         <plugin filename="libgazebo_ros_range.so" name="gazebo_ros_range">
           <topicName>ultrasonic${id}</topicName>
@@ -62,4 +63,5 @@
           <fov>1.0472</fov>
         </plugin>
+        -->
       </sensor>
     </gazebo>

File: antobot_descriptions/antobot_description/urdf/zed2.urdf.xacro (robot description, xacro)
@@ -141,4 +141,5 @@
           </distortion>
         </camera>
+        <!--
         <plugin name="camera_controller" filename="libgazebo_ros_camera.so">
           <robotNamespace>${robot_ns}</robotNamespace>
@@ -157,4 +158,5 @@
           <hackBaseline>0.0</hackBaseline>
         </plugin>
+        -->
       </sensor>
       <sensor type="depth" name="zed2_${position}_left_camera">
@@ -180,4 +182,5 @@
           </noise>
         </camera>
+        <!--
         <plugin name="camera_controller" filename="libgazebo_ros_openni_kinect.so">
           <robotNamespace>${robot_ns}</robotNamespace>
@@ -197,4 +200,5 @@
           <hackBaseline>0.0</hackBaseline>
         </plugin>
+        -->
       </sensor>
     </gazebo>
@@ -231,4 +235,5 @@
           </distortion>
         </camera>
+        <!--
         <plugin name="camera_controller" filename="libgazebo_ros_camera.so">
           <robotNamespace>${robot_ns}</robotNamespace>
@@ -247,4 +252,5 @@
           <hackBaseline>0.12</hackBaseline>
         </plugin>
+        -->
       </sensor>
       <sensor type="camera" name="zed2_${position}_right_camera">
@@ -270,4 +276,5 @@
           </noise>
         </camera>
+        <!--
         <plugin name="camera_controller" filename="libgazebo_ros_camera.so">
           <robotNamespace>${robot_ns}</robotNamespace>
@@ -281,4 +288,5 @@
           <hackBaseline>0.12</hackBaseline>
         </plugin>
+        -->
       </sensor>
     </gazebo>
@@ -287,4 +295,5 @@
       <sensor type="imu" name="zed2_${position}_imu_sensor">
         <update_rate>100</update_rate>
+        <!--
         <plugin filename="libgazebo_ros_imu_sensor.so" name="imu_plugin">
           <robotNamespace>${robot_ns}</robotNamespace>
@@ -294,8 +303,8 @@
           <gaussianNoise>0.01</gaussianNoise>
           <initialOrientationAsReference>false</initialOrientationAsReference>
-          <!-- IMU frame offset copied from an actual ZED2 camera -->
           <xyzOffset>-0.002 -0.023 -0.002</xyzOffset>
           <rpyOffset>0.0014025 -0.0000012 -0.0016915</rpyOffset>
         </plugin>
+        -->
       </sensor>
     </gazebo>
